Commit message: 添加Lider

File: description/robot.urdf.xacro (robot description, xacro)
@@ -2,4 +2,5 @@
 <robot xmlns:xacro="http://www.ros.org/wiki/xacro"  name="robot">
     <xacro:include filename="robot_core.xacro" />
+    <xacro:include filename="lider.xacro" />
     <xacro:include filename="gazebo_control.xacro" />
 </robot>

File: description/robot_core.xacro (robot description, xacro)
@@ -28,4 +28,7 @@
         <material>Gazebo/Black</material>
     </gazebo>
+    <gazebo reference="laser_frame">
+        <material>Gazebo/Red</material>
+    </gazebo>
     <!-- 视觉材质定义 - 用于 RViz 等可视化工具 -->
     <material name="white">
@@ -40,4 +43,7 @@
     <material name="black">
         <color rgba="0 0 0 1"/>
+    </material>
+    <material name="red">
+        <color rgba="1 0 0 1"/>
     </material>
     <!-- ==================== Base Link (基础坐标系) ==================== -->
